File: pcb/eagle/blueimu/blueimu.brd (EAGLE design)
At the start: 50 x 73 mm, 26 parts, among them IC1 ICL7665CPA, IC2 ATMEGA328P, IC3 LP2950Z, J1 22-27-2021-02, Q1 IRL3803, Q2 7.3728MHz

Commit message: Removed unnecessary pull-up resistor from serial line. Added pull-down resistor for LED output.
Parts:
- moved R10 15.5 mm to (24.1, 30.5), turned to 270 degrees
Connections:
- net +3V3: no longer R10.1
- net GND: now also R10.2
- net PD2: now also R10.1
- net TXD: no longer R10.2
Routing:
- net PD2: track 5.94 -> 22.2 mm
- net +3V3: track 169.6 -> 165.2 mm
- net TXD: track 32.7 -> 30.1 mm
Changed lines of the file:
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@@
 </element>
 <element name="C4" library="rcl" package="E2,5-5" value="4.7uF" x="27.94" y="25.4" smashed="yes" rot="R180">
-<attribute name="NAME" x="25.527" y="27.94" size="1.27" layer="25" ratio="10" rot="R180"/>
+<attribute name="NAME" x="29.337" y="29.845" size="1.27" layer="25" ratio="10" rot="R180"/>
 <attribute name="VALUE" x="25.527" y="27.813" size="1.27" layer="27" ratio="10" rot="R180"/>
 </element>
@@
 <element name="U$1" library="gy521" package="GY521" value="GY521" x="13.97" y="62.23" rot="R90"/>
 <element name="U$2" library="hc06" package="HC06" value="HC06" x="11.43" y="31.75" rot="R90"/>
-<element name="R10" library="rcl" package="0207/7" value="10k" x="11.43" y="21.59" smashed="yes" rot="R180">
-<attribute name="NAME" x="13.335" y="22.098" size="1.27" layer="25" ratio="10" rot="R180"/>
-<attribute name="VALUE" x="13.716" y="22.1488" size="1.27" layer="27" ratio="10" rot="R180"/>
+<element name="R10" library="rcl" package="0207/7" value="10k" x="24.13" y="30.48" smashed="yes" rot="R270">
+<attribute name="NAME" x="23.622" y="32.385" size="1.27" layer="25" ratio="10" rot="R270"/>
+<attribute name="VALUE" x="23.5712" y="32.766" size="1.27" layer="27" ratio="10" rot="R270"/>
 </element>
 </elements>
@@
 <contactref element="U$1" pad="ADO"/>
 <contactref element="U$2" pad="KEY"/>
-<via x="15.24" y="41.275" extent="1-16" drill="0.8"/>
+<via x="14.605" y="41.275" extent="1-16" drill="0.8"/>
 <wire x1="14.32" y1="38.85" x2="14.32" y2="40.355" width="0.8128" layer="1"/>
-<wire x1="14.32" y1="40.355" x2="15.24" y2="41.275" width="0.8128" layer="1"/>
+<wire x1="14.32" y1="40.355" x2="14.605" y2="41.275" width="0.8128" layer="1"/>
 <via x="22.86" y="24.13" extent="1-16" drill="0.8"/>
 <wire x1="20.32" y1="24.65" x2="20.84" y2="24.13" width="0.8128" layer="1"/>
 <wire x1="20.84" y1="24.13" x2="22.86" y2="24.13" width="0.8128" layer="1"/>
+<contactref element="R10" pad="2"/>
 </signal>
 <signal name="N$5">
@@
 <wire x1="27.94" y1="54.61" x2="29.21" y2="53.34" width="0.8128" layer="1"/>
 <wire x1="29.21" y1="53.34" x2="29.21" y2="52.07" width="0.8128" layer="1"/>
-<contactref element="R10" pad="1"/>
-<wire x1="15.24" y1="21.59" x2="17.78" y2="21.59" width="0.6096" layer="1"/>
-<wire x1="17.78" y1="21.59" x2="19.05" y2="22.86" width="0.6096" layer="1"/>
 </signal>
 <signal name="TXD">
 <contactref element="IC2" pad="3"/>
-<contactref element="U$2" pad="RX"/>
-<wire x1="3.82" y1="24.65" x2="3.82" y2="22.86" width="0.6096" layer="1"/>
 <wire x1="3.82" y1="22.86" x2="3.81" y2="22.86" width="0.6096" layer="1"/>
 <wire x1="3.81" y1="22.86" x2="5.08" y2="21.59" width="0.6096" layer="1"/>
@@
 <wire x1="13.97" y1="44.45" x2="13.97" y2="43.18" width="0.6096" layer="16"/>
 <wire x1="13.97" y1="43.18" x2="5.08" y2="34.29" width="0.6096" layer="16"/>
-<contactref element="R10" pad="2"/>
-<wire x1="7.62" y1="21.59" x2="5.08" y2="21.59" width="0.6096" layer="1"/>
+<contactref element="U$2" pad="RX"/>
+<wire x1="3.82" y1="24.65" x2="3.81" y2="24.65" width="0.6096" layer="1"/>
+<wire x1="3.81" y1="24.65" x2="3.81" y2="22.86" width="0.6096" layer="1"/>
 </signal>
 <signal name="RXD">
@@
 <contactref element="IC2" pad="4"/>
 <contactref element="U$2" pad="LED"/>
+<contactref element="R10" pad="1"/>
+<wire x1="24.13" y1="34.29" x2="19.05" y2="34.29" width="0.6096" layer="16"/>
+<wire x1="19.05" y1="34.29" x2="16.51" y2="36.83" width="0.6096" layer="16"/>
+<wire x1="16.51" y1="36.83" x2="16.51" y2="44.45" width="0.6096" layer="16"/>
 <wire x1="17.32" y1="38.85" x2="17.32" y2="42.37" width="0.6096" layer="1"/>
 <wire x1="17.32" y1="42.37" x2="16.51" y2="43.18" width="0.6096" layer="1"/>
